Commit message: Adding chlorophyllsensor and test with a randok walk
-> Chlorophyllsensors have been added to the simulation
-> Test setup with a random walk has been added

File: simulation_environment/models/lawn_mower.xacro (robot description, xacro)
@@ -8,5 +8,5 @@
   <!-- Define the chassis -->
   <link name='chassis'>
-    <pose>$0 0 0 0 0 0</pose>
+    <pose>0 0 0 0 0 0</pose>
     <!-- Define inertial system for the chassis -->
     <inertial>
@@ -17,5 +17,5 @@
     <!-- Define collision sorrounding box -->
     <collision name='collision'>
-      <origin xyz="0 0 0" rpy=" 0 0 3.1415"/>
+      <origin xyz="0 0 0" rpy=" 0 0 0"/>
       <geometry>
         <box size="${x_chassis} ${y_chassis} ${z_chassis}"/>
@@ -24,5 +24,5 @@
     <!-- Define visualization structure -->
     <visual name='chassis_visual'>
-	  <origin xyz="0 0 0" rpy=" 0 0 3.1415"/>
+	  <origin xyz="0 0 0" rpy=" 0 0 0"/>
       <geometry>
         <box size="${x_chassis} ${y_chassis} ${z_chassis}"/>
@@ -52,4 +52,17 @@
       </geometry>
     </visual>
+    <!-- Add visual for the chlorophyll sensors. TODO: Change color, make transparent and make a cone -->
+    <visual name='sensor_visual'>
+      <origin xyz="${x_sensor} ${y_sensor} ${-(r_wheel/2+z_chassis/2)/2}" rpy=" 0 0 0"/>
+      <geometry>
+        <cylinder radius="${r_sensor}" length="${r_wheel/2+z_chassis/2}"/>
+      </geometry>
+    </visual>
+    <visual name='sensor_visual'>
+      <origin xyz="${x_sensor} ${-y_sensor} ${-(r_wheel/2+z_chassis/2)/2}" rpy=" 0 0 0"/>
+      <geometry>
+        <cylinder radius="${r_sensor}" length="${r_wheel/2+z_chassis/2}"/>
+      </geometry>
+    </visual>
   </link>
   <!-- Add the wheels for the robot -->
@@ -60,4 +73,14 @@
         <cylinder radius="${r_wheel}" length="${h_wheel}"/>
       </geometry>
+      <surface>
+        <friction>
+          <ode>
+            <mu>0</mu>
+            <mu2>0</mu2>
+            <slip1>1.0</slip1>
+            <slip2>1.0</slip2>
+          </ode>
+        </friction>
+      </surface>
     </collision>
     <visual name="left_wheel_visual">
@@ -70,4 +93,5 @@
       <origin xyz="0 0 0" rpy="0 1.5707 1.5707"/>
       <mass value="${m_wheel}"/>
+      <cylinder_inertia m="${m_wheel}" r="${r_wheel}" h="${h_wheel}"/>
       <xacro:cylinder_inertia m="${m_wheel}" r="${r_wheel}" h="${h_wheel}"/>
     </inertial>
@@ -79,4 +103,14 @@
         <cylinder radius="${r_wheel}" length="${h_wheel}"/>
       </geometry>
+      <surface>
+        <friction>
+          <ode>
+            <mu>0</mu>
+            <mu2>0</mu2>
+            <slip1>1.0</slip1>
+            <slip2>1.0</slip2>
+          </ode>
+        </friction>
+      </surface>
     </collision>
     <visual name="right_wheel_visual">
@@ -89,8 +123,9 @@
       <origin xyz="0 0 0" rpy="0 1.5707 1.5707"/>
       <mass value="${m_wheel}"/>
+      <cylinder_inertia m="${m_wheel}" r="${r_wheel}" h="${h_wheel}"/>
       <xacro:cylinder_inertia m="${m_wheel}" r="${r_wheel}" h="${h_wheel}"/>
     </inertial>
   </link>
-  <!-- TODO: Check if this joint type is correct?-->
+  <!-- Set joints -->
   <joint type="continuous" name="left_wheel_hinge">
     <origin xyz="${-x_chassis/4} ${y_chassis/2+h_wheel/2} ${r_wheel/2-z_chassis/2}" rpy="0 0 0"/>
@@ -106,4 +141,6 @@
     <parent link="chassis"/>
     <axis xyz="0 1 0" rpy="0 0 0"/>
+    <limit effort="100" velocity="100"/>
+    <joint_properties damping="0.0" friction="0.0"/>
   </joint>
-</robot>
+ </robot>

File: simulation_environment/models/parameter.xacro (robot description, xacro)
@@ -2,12 +2,19 @@
 <robot xmlns:xacro="http://www.ros.org/wiki/xacro">
  <!-- Define parameter -->
+  <!-- Parameter for the chassis -->
   <xacro:property name="x_chassis" value="0.5" />
   <xacro:property name="y_chassis" value="0.3" />
   <xacro:property name="z_chassis" value="0.15" />
   <xacro:property name="m_chassis" value="5.0" />
+  <!-- Parameter for the wheels -->
   <xacro:property name="r_wheel" value="0.1075" />
   <xacro:property name="h_wheel" value="0.03" />
-  <xacro:property name="m_wheel" value="0.5" />
-  <xacro:property name="torque_wheel" value="10000" />
+  <!-- TODO: To stable the simulation we had to take a much higher mass value as would be realistic -->
+  <xacro:property name="m_wheel" value="5" />
+  <xacro:property name="torque_wheel" value="100" />
   <xacro:property name="L_wheel" value="0.1788" />
+  <!-- Parameter for the chlorophyll sensors -->
+  <xacro:property name="r_sensor" value="0.01" />
+  <xacro:property name="x_sensor" value="${x_chassis/2 - r_sensor}" />
+  <xacro:property name="y_sensor" value="${y_chassis/2 - r_sensor}" />
 </robot>
