Commit message: Adjusted simulation by adding cameras as Chlorophyllsensors
- Reorganized the structure of the model folder
- Added cameras (1 pixel) as Chlorophyllsensor models
- Added additional Chlorophyll Message and transform node

File: simulation_environment/models/lawn_mower/lawn_mower.xacro (robot description, xacro)
@@ -2,8 +2,8 @@
 <!-- Name the robot -->
 <robot name="lawn_mower" xmlns:xacro="http://www.ros.org/wiki/xacro">
-  <xacro:include filename="$(find simulation_environment)/models/lawn_mower.gazebo" />
-  <xacro:include filename="$(find simulation_environment)/models/materials.xacro" />
-  <xacro:include filename="$(find simulation_environment)/models/macros.xacro" />
-  <xacro:include filename="$(find simulation_environment)/models/parameter.xacro" />
+  <xacro:include filename="$(find simulation_environment)/models/lawn_mower/lawn_mower.gazebo" />
+  <xacro:include filename="$(find simulation_environment)/models/lawn_mower/materials.xacro" />
+  <xacro:include filename="$(find simulation_environment)/models/lawn_mower/macros.xacro" />
+  <xacro:include filename="$(find simulation_environment)/models/lawn_mower/parameter.xacro" />
   <!-- Define the chassis -->
   <link name='chassis'>
@@ -52,18 +52,24 @@
       </geometry>
     </visual>
-    <!-- Add visual for the chlorophyll sensors. TODO: Change color, make transparent and make a cone -->
-    <visual name='sensor_visual'>
-      <origin xyz="${x_sensor} ${y_sensor} ${-(r_wheel/2+z_chassis/2)/2}" rpy=" 0 0 0"/>
-      <geometry>
-        <cylinder radius="${r_sensor}" length="${r_wheel/2+z_chassis/2}"/>
-      </geometry>
-    </visual>
-    <visual name='sensor_visual'>
-      <origin xyz="${x_sensor} ${-y_sensor} ${-(r_wheel/2+z_chassis/2)/2}" rpy=" 0 0 0"/>
-      <geometry>
-        <cylinder radius="${r_sensor}" length="${r_wheel/2+z_chassis/2}"/>
-      </geometry>
-    </visual>
   </link>
+  <!-- Chlorophyllsensors -->
+  <link name="camera_link_1">
+    <xacro:sensor_link_macro l="${l_camera}"/>
+  </link>
+  <joint name="camera_joint_1" type="fixed">
+    <xacro:sensor_joint_macro x="${x_chassis/2 + l_camera/2}" y="${y_chassis/2-l_camera/2}" z="${-z_chassis/2 + l_camera/2}" l="${l_camera}" parent_link="chassis" child_link="camera_link_1"/>
+  </joint>
+  <link name="camera_link_2">
+    <xacro:sensor_link_macro l="${l_camera}"/>
+  </link>
+  <joint name="camera_joint_2" type="fixed">
+    <xacro:sensor_joint_macro x="${x_chassis/2 + l_camera/2}" y="0" z="${-z_chassis/2 + l_camera/2}" l="${l_camera}" parent_link="chassis" child_link="camera_link_2"/>
+  </joint>
+  <link name="camera_link_3">
+    <xacro:sensor_link_macro l="${l_camera}"/>
+  </link>
+  <joint name="camera_joint_3" type="fixed">
+    <xacro:sensor_joint_macro x="${x_chassis/2 + l_camera/2}" y="${-y_chassis/2+l_camera/2}" z="${-z_chassis/2 + l_camera/2}" l="${l_camera}" parent_link="chassis" child_link="camera_link_3"/>
+  </joint>
   <!-- Add the wheels for the robot -->
   <link name="left_wheel">

File: simulation_environment/models/lawn_mower/parameter.xacro (robot description, xacro)
@@ -18,3 +18,5 @@
   <xacro:property name="x_sensor" value="${x_chassis/2 - r_sensor}" />
   <xacro:property name="y_sensor" value="${y_chassis/2 - r_sensor}" />
+  <!-- Camera parameter -->
+  <xacro:property name="l_camera" value="0.02" />
 </robot>

Commit message: Adjust Simulation for Wall Following with one sensor
- Added parameter to choose different number of sensors for simulation
- Added simulation for Wall Following behavior

File: simulation_environment/models/lawn_mower/lawn_mower.xacro (robot description, xacro)
@@ -54,4 +54,13 @@
   </link>
   <!-- Chlorophyllsensors -->
+  <xacro:if value="${$(arg prefix) == 1}">
+	<link name="camera_link">
+		<xacro:sensor_link_macro l="${l_camera}"/>
+	</link>
+	<joint name="camera_joint" type="fixed">
+		<xacro:sensor_joint_macro x="${x_chassis/2 + l_camera/2}" y="0" z="${-z_chassis/2 + l_camera/2}" l="${l_camera}" parent_link="chassis" child_link="camera_link"/>
+	</joint>
+  </xacro:if>
+  <xacro:if value="${$(arg prefix) == 3}">
   <link name="camera_link_1">
     <xacro:sensor_link_macro l="${l_camera}"/>
@@ -72,4 +81,5 @@
     <xacro:sensor_joint_macro x="${x_chassis/2 + l_camera/2}" y="${-y_chassis/2+l_camera/2}" z="${-z_chassis/2 + l_camera/2}" l="${l_camera}" parent_link="chassis" child_link="camera_link_3"/>
   </joint>
+  </xacro:if>
   <!-- Add the wheels for the robot -->
   <link name="left_wheel">

Commit message: Change sensor configurations:
It is now possible to choose between 1,2 or 3 sensors.
The sensor message has changed to mid, left, right signals

File: simulation_environment/models/lawn_mower/lawn_mower.xacro (robot description, xacro)
@@ -55,29 +55,43 @@
   <!-- Chlorophyllsensors -->
   <xacro:if value="${$(arg prefix) == 1}">
-	<link name="camera_link">
+	<link name="camera_link_mid">
 		<xacro:sensor_link_macro l="${l_camera}"/>
 	</link>
-	<joint name="camera_joint" type="fixed">
-		<xacro:sensor_joint_macro x="${x_chassis/2 + l_camera/2}" y="0" z="${-z_chassis/2 + l_camera/2}" l="${l_camera}" parent_link="chassis" child_link="camera_link"/>
+	<joint name="camera_joint_mid" type="fixed">
+		<xacro:sensor_joint_macro x="${x_chassis/2 + l_camera/2}" y="0" z="${-z_chassis/2 + l_camera/2}" l="${l_camera}" parent_link="chassis" child_link="camera_link_mid"/>
 	</joint>
   </xacro:if>
-  <xacro:if value="${$(arg prefix) == 3}">
-  <link name="camera_link_1">
+  <xacro:if value="${$(arg prefix) == 2}">
+  <link name="camera_link_left">
     <xacro:sensor_link_macro l="${l_camera}"/>
   </link>
-  <joint name="camera_joint_1" type="fixed">
-    <xacro:sensor_joint_macro x="${x_chassis/2 + l_camera/2}" y="${y_chassis/2-l_camera/2}" z="${-z_chassis/2 + l_camera/2}" l="${l_camera}" parent_link="chassis" child_link="camera_link_1"/>
+  <joint name="camera_joint_left" type="fixed">
+    <xacro:sensor_joint_macro x="${x_chassis/2 + l_camera/2}" y="${y_chassis/2-l_camera/2}" z="${-z_chassis/2 + l_camera/2}" l="${l_camera}" parent_link="chassis" child_link="camera_link_left"/>
   </joint>
-  <link name="camera_link_2">
+  <link name="camera_link_right">
     <xacro:sensor_link_macro l="${l_camera}"/>
   </link>
-  <joint name="camera_joint_2" type="fixed">
-    <xacro:sensor_joint_macro x="${x_chassis/2 + l_camera/2}" y="0" z="${-z_chassis/2 + l_camera/2}" l="${l_camera}" parent_link="chassis" child_link="camera_link_2"/>
+  <joint name="camera_joint_right" type="fixed">
+    <xacro:sensor_joint_macro x="${x_chassis/2 + l_camera/2}" y="${-y_chassis/2+l_camera/2}" z="${-z_chassis/2 + l_camera/2}" l="${l_camera}" parent_link="chassis" child_link="camera_link_right"/>
   </joint>
-  <link name="camera_link_3">
+  </xacro:if>
+  <xacro:if value="${$(arg prefix) == 3}">
+  <link name="camera_link_left">
     <xacro:sensor_link_macro l="${l_camera}"/>
   </link>
-  <joint name="camera_joint_3" type="fixed">
-    <xacro:sensor_joint_macro x="${x_chassis/2 + l_camera/2}" y="${-y_chassis/2+l_camera/2}" z="${-z_chassis/2 + l_camera/2}" l="${l_camera}" parent_link="chassis" child_link="camera_link_3"/>
+  <joint name="camera_joint_left" type="fixed">
+    <xacro:sensor_joint_macro x="${x_chassis/2 + l_camera/2}" y="${y_chassis/2-l_camera/2}" z="${-z_chassis/2 + l_camera/2}" l="${l_camera}" parent_link="chassis" child_link="camera_link_left"/>
+  </joint>
+  <link name="camera_link_mid">
+    <xacro:sensor_link_macro l="${l_camera}"/>
+  </link>
+  <joint name="camera_joint_mid" type="fixed">
+    <xacro:sensor_joint_macro x="${x_chassis/2 + l_camera/2}" y="0" z="${-z_chassis/2 + l_camera/2}" l="${l_camera}" parent_link="chassis" child_link="camera_link_mid"/>
+  </joint>
+  <link name="camera_link_right">
+    <xacro:sensor_link_macro l="${l_camera}"/>
+  </link>
+  <joint name="camera_joint_right" type="fixed">
+    <xacro:sensor_joint_macro x="${x_chassis/2 + l_camera/2}" y="${-y_chassis/2+l_camera/2}" z="${-z_chassis/2 + l_camera/2}" l="${l_camera}" parent_link="chassis" child_link="camera_link_right"/>
   </joint>
   </xacro:if>

File: simulation_environment/models/lawn_mower/parameter.xacro (robot description, xacro)
@@ -2,21 +2,20 @@
 <robot xmlns:xacro="http://www.ros.org/wiki/xacro">
  <!-- Define parameter -->
+  <!-- load parameters from yaml file -->
+  <xacro:property name="yaml_file" 		value="$(find simulation_environment)/config/props.yaml" />
+  <xacro:property name="props" 			value="${load_yaml(yaml_file)}"/>
   <!-- Parameter for the chassis -->
-  <xacro:property name="x_chassis" value="0.5" />
-  <xacro:property name="y_chassis" value="0.3" />
-  <xacro:property name="z_chassis" value="0.15" />
-  <xacro:property name="m_chassis" value="5.0" />
+  <xacro:property name="x_chassis" 		value="${props['x_chassis']}" />
+  <xacro:property name="y_chassis" 		value="${props['y_chassis']}" />
+  <xacro:property name="z_chassis" 		value="${props['z_chassis']}" />
+  <xacro:property name="m_chassis" 		value="${props['m_chassis']}" />
   <!-- Parameter for the wheels -->
-  <xacro:property name="r_wheel" value="0.1075" />
-  <xacro:property name="h_wheel" value="0.03" />
+  <xacro:property name="r_wheel" 		value="${props['r_wheel']}" />
+  <xacro:property name="h_wheel" 		value="${props['h_wheel']}" />
+  <xacro:property name="L_wheel" 		value="${props['L_wheel']}" />
   <!-- TODO: To stable the simulation we had to take a much higher mass value as would be realistic -->
-  <xacro:property name="m_wheel" value="5" />
-  <xacro:property name="torque_wheel" value="100" />
-  <xacro:property name="L_wheel" value="0.1788" />
-  <!-- Parameter for the chlorophyll sensors -->
-  <xacro:property name="r_sensor" value="0.01" />
-  <xacro:property name="x_sensor" value="${x_chassis/2 - r_sensor}" />
-  <xacro:property name="y_sensor" value="${y_chassis/2 - r_sensor}" />
+  <xacro:property name="m_wheel" 		value="5" />
+  <xacro:property name="torque_wheel" 	value="100" />
   <!-- Camera parameter -->
-  <xacro:property name="l_camera" value="0.02" />
+  <xacro:property name="l_camera" 		value="${props['l_camera']}" />
 </robot>

Commit message: Fixed Problems: - Map generation - Odometry Error - added PGO and LC visualization
Open:
- Include noise to odometry data

File: simulation_environment/models/lawn_mower/lawn_mower.xacro (robot description, xacro)
@@ -53,4 +53,24 @@
     </visual>
   </link>
+   <!-- Add an odom link -->
+  <link name="odom_link" >
+	<collision>
+      <origin xyz="0 0 0" rpy="0 0 0"/>
+      <geometry>
+		<box size="1e-6 1e-6 1e-6"/>
+      </geometry>
+    </collision>
+    <inertial>
+      <mass value="1e-5" />
+      <origin xyz="0 0 0" rpy="0 0 0"/>
+      <inertia ixx="1e-6" ixy="0" ixz="0" iyy="1e-6" iyz="0" izz="1e-6" />
+    </inertial>
+  </link>
+  <joint name="odom_joint" type="fixed">
+    <axis xyz="0 1 0" />
+    <origin xyz="${-X_wheel} 0 0" rpy="0 0 0"/>
+    <parent link="chassis"/>
+    <child link="odom_link"/>
+  </joint>
   <!-- Chlorophyllsensors -->
   <xacro:if value="${$(arg prefix) == 1}">
@@ -106,8 +126,8 @@
         <friction>
           <ode>
-            <mu>0</mu>
-            <mu2>0</mu2>
-            <slip1>1.0</slip1>
-            <slip2>1.0</slip2>
+            <mu>100.0</mu>
+            <mu2>100.0</mu2>
+            <slip1>0.0</slip1>
+            <slip2>0.0</slip2>
           </ode>
         </friction>
@@ -136,8 +156,8 @@
         <friction>
           <ode>
-            <mu>0</mu>
-            <mu2>0</mu2>
-            <slip1>1.0</slip1>
-            <slip2>1.0</slip2>
+            <mu>100.0</mu>
+            <mu2>100.0</mu2>
+            <slip1>0.0</slip1>
+            <slip2>0.0</slip2>
           </ode>
         </friction>
@@ -159,7 +179,7 @@
   <!-- Set joints -->
   <joint type="continuous" name="left_wheel_hinge">
-    <origin xyz="${-x_chassis/4} ${y_chassis/2+h_wheel/2} ${r_wheel/2-z_chassis/2}" rpy="0 0 0"/>
+    <origin xyz="0 ${L_wheel} ${r_wheel/2-z_chassis/2}" rpy="0 0 0"/>
     <child link="left_wheel"/>
-    <parent link="chassis"/>
+    <parent link="odom_link"/>
     <axis xyz="0 1 0" rpy="0 0 0"/>
     <limit effort="100" velocity="100"/>
@@ -167,7 +187,7 @@
   </joint>
   <joint type="continuous" name="right_wheel_hinge">
-    <origin xyz="${-x_chassis/4} ${-y_chassis/2-h_wheel/2} ${r_wheel/2-z_chassis/2}" rpy="0 0 0"/>
+    <origin xyz="0 ${-L_wheel} ${r_wheel/2-z_chassis/2}" rpy="0 0 0"/>
     <child link="right_wheel"/>
-    <parent link="chassis"/>
+    <parent link="odom_link"/>
     <axis xyz="0 1 0" rpy="0 0 0"/>
     <limit effort="100" velocity="100"/>

File: simulation_environment/models/lawn_mower/parameter.xacro (robot description, xacro)
@@ -14,7 +14,7 @@
   <xacro:property name="h_wheel" 		value="${props['h_wheel']}" />
   <xacro:property name="L_wheel" 		value="${props['L_wheel']}" />
-  <!-- TODO: To stable the simulation we had to take a much higher mass value as would be realistic -->
-  <xacro:property name="m_wheel" 		value="5" />
-  <xacro:property name="torque_wheel" 	value="100" />
+  <xacro:property name="X_wheel"		value="${props['X_wheel']}" />
+  <xacro:property name="m_wheel" 		value="${props['m_wheel']}" />
+  <xacro:property name="torque_wheel" 	value="${props['torque_wheel']}" />
   <!-- Camera parameter -->
   <xacro:property name="l_camera" 		value="${props['l_camera']}" />
